File: LandstromWarnung.sch (KiCad schematic (older format))
At the start: 19 parts, among them J10 K15 -, J11 Summer +, J3 Summer -, J7 Landstr. +, J8 Landstr. -, J9 K15 +, Q2 IRF7404, U5 LTV-847

Commit message: x
Parts:
- gave numbers to parts that had none: 2
Changed lines of the file:
@@
 $EndComp
 $Comp
-L Device:Polyfuse F?
+L Device:Polyfuse F1
 U 1 1 60411390
 P 7455 3200
-F 0 "F?" V 7230 3200 50  0000 C CNN
+F 0 "F1" V 7230 3200 50  0000 C CNN
 F 1 "Polyfuse" V 7321 3200 50  0000 C CNN
 F 2 "Resistor_SMD:R_0603_1608Metric_Pad1.05x0.95mm_HandSolder" H 7505 3000 50  0001 L CNN
@@
 $EndComp
 $Comp
-L Device:Polyfuse F?
+L Device:Polyfuse F2
 U 1 1 60413092
 P 7755 3745
-F 0 "F?" V 7530 3745 50  0000 C CNN
+F 0 "F2" V 7530 3745 50  0000 C CNN
 F 1 "Polyfuse" V 7621 3745 50  0000 C CNN
 F 2 "Resistor_SMD:R_0603_1608Metric_Pad1.05x0.95mm_HandSolder" H 7805 3545 50  0001 L CNN
